File: minimal_ad74416h_stack_adapter/minimal_ad74416h_stack_adapter.kicad_pcb (KiCad board)
At the start: 2 copper layers, 5.1 x 5.1 mm, 0 parts

Commit message: backup
Parts:
- added J1: CLP-133-02-G-D-BE, connector_footprints:CLP-133-02-G-D-BE, F.Cu at (139.7, 106.2)
- added J2: CLP-133-02-G-D-BE, connector_footprints:CLP-133-02-G-D-BE, F.Cu at (139.7, 118.4)
- added J3: CLP-133-02-G-D-BE, connector_footprints:CLP-133-02-G-D-BE, F.Cu at (139.7, 124.5)
- added J4: CLP-133-02-G-D-BE, connector_footprints:CLP-133-02-G-D-BE, F.Cu at (139.7, 130.6)
- added J5: CLP-133-02-G-D-BE, connector_footprints:CLP-133-02-G-D-BE, F.Cu at (139.7, 142.7)
Other:
- board size 5.1 x 5.1 mm -> 45.7 x 45.7 mm
- copper layers 2 -> 4

Commit message: backup
Parts:
- added J6: FW-33-03-G-D-085-155, connector_footprints:FW-33-03-G-D-085-155, F.Cu at (139.7, 99.2)
Other:
- board size 45.7 x 45.7 mm -> 45.7 x 53.3 mm

Commit message: backup
Parts:
- removed the J3 at (139.7, 124.5)
- renumbered J6 to J1, J1 to J2, J2 to J3
Connections:
- J1 pad 1: unconnected-(J6-Pad1) -> GNDA
- J1 pad 10: unconnected-(J6-Pad10) -> /SDO
- J1 pad 11: unconnected-(J6-Pad11) -> /SDI
- J1 pad 12: unconnected-(J6-Pad12) -> /SDI
- J1 pad 13: unconnected-(J6-Pad13) -> /SCLK
- J1 pad 14: unconnected-(J6-Pad14) -> /SCLK
- J1 pad 15: unconnected-(J6-Pad15) -> /2B4
- J1 pad 16: unconnected-(J6-Pad16) -> /2B4
- J1 pad 17: unconnected-(J6-Pad17) -> /2B3
- J1 pad 18: unconnected-(J6-Pad18) -> /2B3
- J1 pad 19: unconnected-(J6-Pad19) -> /2B2
- J1 pad 2: unconnected-(J6-Pad2) -> GNDA
- J1 pad 20: unconnected-(J6-Pad20) -> /2B2
- J1 pad 21: unconnected-(J6-Pad21) -> /2B1
- J1 pad 22: unconnected-(J6-Pad22) -> /2B1
- J1 pad 23: unconnected-(J6-Pad23) -> /1B4
- J1 pad 24: unconnected-(J6-Pad24) -> /1B4
- J1 pad 25: unconnected-(J6-Pad25) -> /1B3
- J1 pad 26: unconnected-(J6-Pad26) -> /1B3
- J1 pad 27: unconnected-(J6-Pad27) -> /1B2
- J1 pad 28: unconnected-(J6-Pad28) -> /1B2
- J1 pad 29: unconnected-(J6-Pad29) -> /1B1
- J1 pad 3: unconnected-(J6-Pad3) -> /24V0
- J1 pad 30: unconnected-(J6-Pad30) -> /1B1
- J1 pad 31: unconnected-(J6-Pad31) -> GNDA
- J1 pad 32: unconnected-(J6-Pad32) -> GNDA
- J1 pad 33: unconnected-(J6-Pad33) -> /3V3
- J1 pad 34: unconnected-(J6-Pad34) -> /3V3
- J1 pad 35: unconnected-(J6-Pad35) -> GNDA
- J1 pad 36: unconnected-(J6-Pad36) -> GNDA
- J1 pad 37: unconnected-(J6-Pad37) -> GNDA
- J1 pad 38: unconnected-(J6-Pad38) -> GNDA
- J1 pad 39: unconnected-(J6-Pad39) -> /-15V0
- J1 pad 4: unconnected-(J6-Pad4) -> /24V0
- J1 pad 40: unconnected-(J6-Pad40) -> /-15V0
- J1 pad 41: unconnected-(J6-Pad41) -> GNDA
- J1 pad 42: unconnected-(J6-Pad42) -> GNDA
- J1 pad 43: unconnected-(J6-Pad43) -> GNDA
- J1 pad 44: unconnected-(J6-Pad44) -> GNDA
- J1 pad 45: unconnected-(J6-Pad45) -> /5V0
- J1 pad 46: unconnected-(J6-Pad46) -> /5V0
- J1 pad 47: unconnected-(J6-Pad47) -> GNDA
- J1 pad 48: unconnected-(J6-Pad48) -> GNDA
- J1 pad 49: unconnected-(J6-Pad49) -> /SCL
- J1 pad 5: unconnected-(J6-Pad5) -> GNDA
- J1 pad 50: unconnected-(J6-Pad50) -> /SCL
- J1 pad 51: unconnected-(J6-Pad51) -> /SDA
- J1 pad 52: unconnected-(J6-Pad52) -> /SDA
- J1 pad 53: unconnected-(J6-Pad53) -> GNDA
- J1 pad 54: unconnected-(J6-Pad54) -> GNDA
- J1 pad 55: unconnected-(J6-Pad55) -> GNDA
- J1 pad 56: unconnected-(J6-Pad56) -> GNDA
- J1 pad 57: unconnected-(J6-Pad57) -> /DO_VDD
- J1 pad 58: unconnected-(J6-Pad58) -> /DO_VDD
- J1 pad 59: unconnected-(J6-Pad59) -> GNDA
- J1 pad 6: unconnected-(J6-Pad6) -> GNDA
- J1 pad 60: unconnected-(J6-Pad60) -> GNDA
- J1 pad 61: unconnected-(J6-Pad61) -> GNDA
- J1 pad 62: unconnected-(J6-Pad62) -> GNDA
- J1 pad 63: unconnected-(J6-Pad63) -> /14V5
- J1 pad 64: unconnected-(J6-Pad64) -> /14V5
- J1 pad 65: unconnected-(J6-Pad65) -> GNDA
- J1 pad 66: unconnected-(J6-Pad66) -> GNDA
- J1 pad 7: unconnected-(J6-Pad7) -> /~{SYNC}
- J1 pad 8: unconnected-(J6-Pad8) -> /~{SYNC}
- J1 pad 9: unconnected-(J6-Pad9) -> /SDO
- J2 pad 1: unconnected-(J1-Pad1) -> GNDA
- J2 pad 10: unconnected-(J1-Pad10) -> /SDO
- J2 pad 11: unconnected-(J1-Pad11) -> /SDI
- J2 pad 12: unconnected-(J1-Pad12) -> /SDI
- J2 pad 13: unconnected-(J1-Pad13) -> /SCLK
- J2 pad 14: unconnected-(J1-Pad14) -> /SCLK
- J2 pad 15: unconnected-(J1-Pad15) -> /2B4
- J2 pad 16: unconnected-(J1-Pad16) -> /2B4
- J2 pad 17: unconnected-(J1-Pad17) -> /2B3
- J2 pad 18: unconnected-(J1-Pad18) -> /2B3
- J2 pad 19: unconnected-(J1-Pad19) -> /2B2
- J2 pad 2: unconnected-(J1-Pad2) -> GNDA
- J2 pad 20: unconnected-(J1-Pad20) -> /2B2
- J2 pad 21: unconnected-(J1-Pad21) -> /2B1
- J2 pad 22: unconnected-(J1-Pad22) -> /2B1
- J2 pad 23: unconnected-(J1-Pad23) -> /1B4
- J2 pad 24: unconnected-(J1-Pad24) -> /1B4
- J2 pad 25: unconnected-(J1-Pad25) -> /1B3
- J2 pad 26: unconnected-(J1-Pad26) -> /1B3
- J2 pad 27: unconnected-(J1-Pad27) -> /1B2
- J2 pad 28: unconnected-(J1-Pad28) -> /1B2
- J2 pad 29: unconnected-(J1-Pad29) -> /1B1
- J2 pad 3: unconnected-(J1-Pad3) -> /24V0
- J2 pad 30: unconnected-(J1-Pad30) -> /1B1
- J2 pad 31: unconnected-(J1-Pad31) -> GNDA
- J2 pad 32: unconnected-(J1-Pad32) -> GNDA
- J2 pad 33: unconnected-(J1-Pad33) -> /3V3
- J2 pad 34: unconnected-(J1-Pad34) -> /3V3
- J2 pad 35: unconnected-(J1-Pad35) -> GNDA
- J2 pad 36: unconnected-(J1-Pad36) -> GNDA
- J2 pad 37: unconnected-(J1-Pad37) -> GNDA
- J2 pad 38: unconnected-(J1-Pad38) -> GNDA
- J2 pad 39: unconnected-(J1-Pad39) -> /-15V0
- J2 pad 4: unconnected-(J1-Pad4) -> /24V0
- J2 pad 40: unconnected-(J1-Pad40) -> /-15V0
- J2 pad 41: unconnected-(J1-Pad41) -> GNDA
- J2 pad 42: unconnected-(J1-Pad42) -> GNDA
- J2 pad 43: unconnected-(J1-Pad43) -> GNDA
- J2 pad 44: unconnected-(J1-Pad44) -> GNDA
- J2 pad 45: unconnected-(J1-Pad45) -> /5V0
- J2 pad 46: unconnected-(J1-Pad46) -> /5V0
- J2 pad 47: unconnected-(J1-Pad47) -> GNDA
- J2 pad 48: unconnected-(J1-Pad48) -> GNDA
- J2 pad 49: unconnected-(J1-Pad49) -> /SCL
- J2 pad 5: unconnected-(J1-Pad5) -> GNDA
- J2 pad 50: unconnected-(J1-Pad50) -> /SCL
- J2 pad 51: unconnected-(J1-Pad51) -> /SDA
- J2 pad 52: unconnected-(J1-Pad52) -> /SDA
- J2 pad 53: unconnected-(J1-Pad53) -> GNDA
- J2 pad 54: unconnected-(J1-Pad54) -> GNDA
- J2 pad 55: unconnected-(J1-Pad55) -> GNDA
- J2 pad 56: unconnected-(J1-Pad56) -> GNDA
- J2 pad 57: unconnected-(J1-Pad57) -> /DO_VDD
- J2 pad 58: unconnected-(J1-Pad58) -> /DO_VDD
- J2 pad 59: unconnected-(J1-Pad59) -> GNDA
- J2 pad 6: unconnected-(J1-Pad6) -> GNDA
- J2 pad 60: unconnected-(J1-Pad60) -> GNDA
- J2 pad 61: unconnected-(J1-Pad61) -> GNDA
- J2 pad 62: unconnected-(J1-Pad62) -> GNDA
- J2 pad 63: unconnected-(J1-Pad63) -> /14V5
- J2 pad 64: unconnected-(J1-Pad64) -> /14V5
- J2 pad 65: unconnected-(J1-Pad65) -> GNDA
- J2 pad 66: unconnected-(J1-Pad66) -> GNDA
- J2 pad 7: unconnected-(J1-Pad7) -> /~{SYNC}
- J2 pad 8: unconnected-(J1-Pad8) -> /~{SYNC}
- J2 pad 9: unconnected-(J1-Pad9) -> /SDO
- J3 pad 1: unconnected-(J2-Pad1) -> GNDA
- J3 pad 10: unconnected-(J2-Pad10) -> /SDO
- J3 pad 11: unconnected-(J2-Pad11) -> /SDI
- J3 pad 12: unconnected-(J2-Pad12) -> /SDI
- J3 pad 13: unconnected-(J2-Pad13) -> /SCLK
- J3 pad 14: unconnected-(J2-Pad14) -> /SCLK
- J3 pad 15: unconnected-(J2-Pad15) -> /2B4
- J3 pad 16: unconnected-(J2-Pad16) -> /2B4
- J3 pad 17: unconnected-(J2-Pad17) -> /2B3
- J3 pad 18: unconnected-(J2-Pad18) -> /2B3
- J3 pad 19: unconnected-(J2-Pad19) -> /2B2
- J3 pad 2: unconnected-(J2-Pad2) -> GNDA
- J3 pad 20: unconnected-(J2-Pad20) -> /2B2
- J3 pad 21: unconnected-(J2-Pad21) -> /2B1
- J3 pad 22: unconnected-(J2-Pad22) -> /2B1
- J3 pad 23: unconnected-(J2-Pad23) -> /1B4
- J3 pad 24: unconnected-(J2-Pad24) -> /1B4
- J3 pad 25: unconnected-(J2-Pad25) -> /1B3
- J3 pad 26: unconnected-(J2-Pad26) -> /1B3
- J3 pad 27: unconnected-(J2-Pad27) -> /1B2
- J3 pad 28: unconnected-(J2-Pad28) -> /1B2
- J3 pad 29: unconnected-(J2-Pad29) -> /1B1
- J3 pad 3: unconnected-(J2-Pad3) -> /24V0
- J3 pad 30: unconnected-(J2-Pad30) -> /1B1
- J3 pad 31: unconnected-(J2-Pad31) -> GNDA
- J3 pad 32: unconnected-(J2-Pad32) -> GNDA
- J3 pad 33: unconnected-(J2-Pad33) -> /3V3
- J3 pad 34: unconnected-(J2-Pad34) -> /3V3
- J3 pad 35: unconnected-(J2-Pad35) -> GNDA
- J3 pad 36: unconnected-(J2-Pad36) -> GNDA
- J3 pad 37: unconnected-(J2-Pad37) -> GNDA
- J3 pad 38: unconnected-(J2-Pad38) -> GNDA
- J3 pad 39: unconnected-(J2-Pad39) -> /-15V0
- J3 pad 4: unconnected-(J2-Pad4) -> /24V0
- J3 pad 40: unconnected-(J2-Pad40) -> /-15V0
- J3 pad 41: unconnected-(J2-Pad41) -> GNDA
- J3 pad 42: unconnected-(J2-Pad42) -> GNDA
- J3 pad 43: unconnected-(J2-Pad43) -> GNDA
- J3 pad 44: unconnected-(J2-Pad44) -> GNDA
- J3 pad 45: unconnected-(J2-Pad45) -> /5V0
- J3 pad 46: unconnected-(J2-Pad46) -> /5V0
- J3 pad 47: unconnected-(J2-Pad47) -> GNDA
- J3 pad 48: unconnected-(J2-Pad48) -> GNDA
- J3 pad 49: unconnected-(J2-Pad49) -> /SCL
- J3 pad 5: unconnected-(J2-Pad5) -> GNDA
- J3 pad 50: unconnected-(J2-Pad50) -> /SCL
- J3 pad 51: unconnected-(J2-Pad51) -> /SDA
- J3 pad 52: unconnected-(J2-Pad52) -> /SDA
- J3 pad 53: unconnected-(J2-Pad53) -> GNDA
- J3 pad 54: unconnected-(J2-Pad54) -> GNDA
- J3 pad 55: unconnected-(J2-Pad55) -> GNDA
- J3 pad 56: unconnected-(J2-Pad56) -> GNDA
- J3 pad 57: unconnected-(J2-Pad57) -> /DO_VDD
- J3 pad 58: unconnected-(J2-Pad58) -> /DO_VDD
- J3 pad 59: unconnected-(J2-Pad59) -> GNDA
- J3 pad 6: unconnected-(J2-Pad6) -> GNDA
- J3 pad 60: unconnected-(J2-Pad60) -> GNDA
- J3 pad 61: unconnected-(J2-Pad61) -> GNDA
- J3 pad 62: unconnected-(J2-Pad62) -> GNDA
- J3 pad 63: unconnected-(J2-Pad63) -> /14V5
- J3 pad 64: unconnected-(J2-Pad64) -> /14V5
- J3 pad 65: unconnected-(J2-Pad65) -> GNDA
- J3 pad 66: unconnected-(J2-Pad66) -> GNDA
- J3 pad 7: unconnected-(J2-Pad7) -> /~{SYNC}
- J3 pad 8: unconnected-(J2-Pad8) -> /~{SYNC}
- J3 pad 9: unconnected-(J2-Pad9) -> /SDO
- J4 pad 1: unconnected-(J4-Pad1) -> GNDA
- J4 pad 10: unconnected-(J4-Pad10) -> /SDO
- J4 pad 11: unconnected-(J4-Pad11) -> /SDI
- J4 pad 12: unconnected-(J4-Pad12) -> /SDI
- J4 pad 13: unconnected-(J4-Pad13) -> /SCLK
- J4 pad 14: unconnected-(J4-Pad14) -> /SCLK
- J4 pad 15: unconnected-(J4-Pad15) -> /2B4
- J4 pad 16: unconnected-(J4-Pad16) -> /2B4
- J4 pad 17: unconnected-(J4-Pad17) -> /2B3
- J4 pad 18: unconnected-(J4-Pad18) -> /2B3
- J4 pad 19: unconnected-(J4-Pad19) -> /2B2
- J4 pad 2: unconnected-(J4-Pad2) -> GNDA
- J4 pad 20: unconnected-(J4-Pad20) -> /2B2
- J4 pad 21: unconnected-(J4-Pad21) -> /2B1
- J4 pad 22: unconnected-(J4-Pad22) -> /2B1
- J4 pad 23: unconnected-(J4-Pad23) -> /1B4
- J4 pad 24: unconnected-(J4-Pad24) -> /1B4
- J4 pad 25: unconnected-(J4-Pad25) -> /1B3
- J4 pad 26: unconnected-(J4-Pad26) -> /1B3
- J4 pad 27: unconnected-(J4-Pad27) -> /1B2
- J4 pad 28: unconnected-(J4-Pad28) -> /1B2
- J4 pad 29: unconnected-(J4-Pad29) -> /1B1
- J4 pad 3: unconnected-(J4-Pad3) -> /24V0
- J4 pad 30: unconnected-(J4-Pad30) -> /1B1
- J4 pad 31: unconnected-(J4-Pad31) -> GNDA
- J4 pad 32: unconnected-(J4-Pad32) -> GNDA
- J4 pad 33: unconnected-(J4-Pad33) -> /3V3
- J4 pad 34: unconnected-(J4-Pad34) -> /3V3
- J4 pad 35: unconnected-(J4-Pad35) -> GNDA
- J4 pad 36: unconnected-(J4-Pad36) -> GNDA
- J4 pad 37: unconnected-(J4-Pad37) -> GNDA
- J4 pad 38: unconnected-(J4-Pad38) -> GNDA
- J4 pad 39: unconnected-(J4-Pad39) -> /-15V0
- J4 pad 4: unconnected-(J4-Pad4) -> /24V0
- J4 pad 40: unconnected-(J4-Pad40) -> /-15V0
- J4 pad 41: unconnected-(J4-Pad41) -> GNDA
- J4 pad 42: unconnected-(J4-Pad42) -> GNDA
- J4 pad 43: unconnected-(J4-Pad43) -> GNDA
- J4 pad 44: unconnected-(J4-Pad44) -> GNDA
- J4 pad 45: unconnected-(J4-Pad45) -> /5V0
- J4 pad 46: unconnected-(J4-Pad46) -> /5V0
- J4 pad 47: unconnected-(J4-Pad47) -> GNDA
- J4 pad 48: unconnected-(J4-Pad48) -> GNDA
- J4 pad 49: unconnected-(J4-Pad49) -> /SCL
- J4 pad 5: unconnected-(J4-Pad5) -> GNDA
- J4 pad 50: unconnected-(J4-Pad50) -> /SCL
- J4 pad 51: unconnected-(J4-Pad51) -> /SDA
- J4 pad 52: unconnected-(J4-Pad52) -> /SDA
- J4 pad 53: unconnected-(J4-Pad53) -> GNDA
- J4 pad 54: unconnected-(J4-Pad54) -> GNDA
- J4 pad 55: unconnected-(J4-Pad55) -> GNDA
- J4 pad 56: unconnected-(J4-Pad56) -> GNDA
- J4 pad 57: unconnected-(J4-Pad57) -> /DO_VDD
- J4 pad 58: unconnected-(J4-Pad58) -> /DO_VDD
- J4 pad 59: unconnected-(J4-Pad59) -> GNDA
- J4 pad 6: unconnected-(J4-Pad6) -> GNDA
- J4 pad 60: unconnected-(J4-Pad60) -> GNDA
- J4 pad 61: unconnected-(J4-Pad61) -> GNDA
- J4 pad 62: unconnected-(J4-Pad62) -> GNDA
- J4 pad 63: unconnected-(J4-Pad63) -> /14V5
- J4 pad 64: unconnected-(J4-Pad64) -> /14V5
- J4 pad 65: unconnected-(J4-Pad65) -> GNDA
- J4 pad 66: unconnected-(J4-Pad66) -> GNDA
- J4 pad 7: unconnected-(J4-Pad7) -> /~{SYNC}
- J4 pad 8: unconnected-(J4-Pad8) -> /~{SYNC}
- J4 pad 9: unconnected-(J4-Pad9) -> /SDO
- J5 pad 1: unconnected-(J5-Pad1) -> GNDA
- J5 pad 10: unconnected-(J5-Pad10) -> /SDO
- J5 pad 11: unconnected-(J5-Pad11) -> /SDI
- J5 pad 12: unconnected-(J5-Pad12) -> /SDI
- J5 pad 13: unconnected-(J5-Pad13) -> /SCLK
- J5 pad 14: unconnected-(J5-Pad14) -> /SCLK
- J5 pad 15: unconnected-(J5-Pad15) -> /2B4
- J5 pad 16: unconnected-(J5-Pad16) -> /2B4
- J5 pad 17: unconnected-(J5-Pad17) -> /2B3
- J5 pad 18: unconnected-(J5-Pad18) -> /2B3
- J5 pad 19: unconnected-(J5-Pad19) -> /2B2
- J5 pad 2: unconnected-(J5-Pad2) -> GNDA
- J5 pad 20: unconnected-(J5-Pad20) -> /2B2
- J5 pad 21: unconnected-(J5-Pad21) -> /2B1
- J5 pad 22: unconnected-(J5-Pad22) -> /2B1
- J5 pad 23: unconnected-(J5-Pad23) -> /1B4
- J5 pad 24: unconnected-(J5-Pad24) -> /1B4
- J5 pad 25: unconnected-(J5-Pad25) -> /1B3
- J5 pad 26: unconnected-(J5-Pad26) -> /1B3
- J5 pad 27: unconnected-(J5-Pad27) -> /1B2
- J5 pad 28: unconnected-(J5-Pad28) -> /1B2
- J5 pad 29: unconnected-(J5-Pad29) -> /1B1
- J5 pad 3: unconnected-(J5-Pad3) -> /24V0
- J5 pad 30: unconnected-(J5-Pad30) -> /1B1
- J5 pad 31: unconnected-(J5-Pad31) -> GNDA
- J5 pad 32: unconnected-(J5-Pad32) -> GNDA
- J5 pad 33: unconnected-(J5-Pad33) -> /3V3
- J5 pad 34: unconnected-(J5-Pad34) -> /3V3
- J5 pad 35: unconnected-(J5-Pad35) -> GNDA
- J5 pad 36: unconnected-(J5-Pad36) -> GNDA
- J5 pad 37: unconnected-(J5-Pad37) -> GNDA
- J5 pad 38: unconnected-(J5-Pad38) -> GNDA
- J5 pad 39: unconnected-(J5-Pad39) -> /-15V0
- J5 pad 4: unconnected-(J5-Pad4) -> /24V0
- J5 pad 40: unconnected-(J5-Pad40) -> /-15V0
- J5 pad 41: unconnected-(J5-Pad41) -> GNDA
- J5 pad 42: unconnected-(J5-Pad42) -> GNDA
- J5 pad 43: unconnected-(J5-Pad43) -> GNDA
- J5 pad 44: unconnected-(J5-Pad44) -> GNDA
- J5 pad 45: unconnected-(J5-Pad45) -> /5V0
- J5 pad 46: unconnected-(J5-Pad46) -> /5V0
- J5 pad 47: unconnected-(J5-Pad47) -> GNDA
- J5 pad 48: unconnected-(J5-Pad48) -> GNDA
- J5 pad 49: unconnected-(J5-Pad49) -> /SCL
- J5 pad 5: unconnected-(J5-Pad5) -> GNDA
- J5 pad 50: unconnected-(J5-Pad50) -> /SCL
- J5 pad 51: unconnected-(J5-Pad51) -> /SDA
- J5 pad 52: unconnected-(J5-Pad52) -> /SDA
- J5 pad 53: unconnected-(J5-Pad53) -> GNDA
- J5 pad 54: unconnected-(J5-Pad54) -> GNDA
- J5 pad 55: unconnected-(J5-Pad55) -> GNDA
- J5 pad 56: unconnected-(J5-Pad56) -> GNDA
- J5 pad 57: unconnected-(J5-Pad57) -> /DO_VDD
- J5 pad 58: unconnected-(J5-Pad58) -> /DO_VDD
- J5 pad 59: unconnected-(J5-Pad59) -> GNDA
- J5 pad 6: unconnected-(J5-Pad6) -> GNDA
- J5 pad 60: unconnected-(J5-Pad60) -> GNDA
- J5 pad 61: unconnected-(J5-Pad61) -> GNDA
- J5 pad 62: unconnected-(J5-Pad62) -> GNDA
- J5 pad 63: unconnected-(J5-Pad63) -> /14V5
- J5 pad 64: unconnected-(J5-Pad64) -> /14V5
- J5 pad 65: unconnected-(J5-Pad65) -> GNDA
- J5 pad 66: unconnected-(J5-Pad66) -> GNDA
- J5 pad 7: unconnected-(J5-Pad7) -> /~{SYNC}
- J5 pad 8: unconnected-(J5-Pad8) -> /~{SYNC}
- J5 pad 9: unconnected-(J5-Pad9) -> /SDO
Routing:
- net /2B3: track 0.00 -> 60.7 mm, vias 0 -> 8
- net /~{SYNC}: track 0.00 -> 60.7 mm, vias 0 -> 8
- net /SCLK: track 0.00 -> 60.7 mm, vias 0 -> 8
- net /2B1: track 0.00 -> 60.7 mm, vias 0 -> 8
- net /1B2: track 0.00 -> 60.7 mm, vias 0 -> 8
- net /SDO: track 0.00 -> 60.7 mm, vias 0 -> 8
- net /1B3: track 0.00 -> 60.7 mm, vias 0 -> 8
- net /SCL: track 0.00 -> 60.7 mm, vias 0 -> 8
- net /1B4: track 0.00 -> 60.7 mm, vias 0 -> 8
- net /SDA: track 0.00 -> 60.7 mm, vias 0 -> 8
- net /1B1: track 0.00 -> 60.7 mm, vias 0 -> 8
- net /SDI: track 0.00 -> 60.7 mm, vias 0 -> 8
- net /2B4: track 0.00 -> 60.7 mm, vias 0 -> 8
- net /2B2: track 0.00 -> 60.6 mm, vias 0 -> 8
- net GNDA: vias 0 -> 104
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- added copper zone on F.Cu, net /-15V0
- added copper zone on In1.Cu, net /-15V0
- added copper zone on F.Cu, net /14V5
- added copper zone on In1.Cu, net /14V5
- added copper zone on F.Cu, net /24V0
- added copper zone on In1.Cu, net /24V0
- added copper zone on F.Cu, net /3V3
- added copper zone on In1.Cu, net /3V3
- added copper zone on F.Cu, net /5V0
- added copper zone on In1.Cu, net /5V0
- added copper zone on F.Cu, net /DO_VDD
- added copper zone on In1.Cu, net /DO_VDD
- added copper zone on B.Cu, net GNDA
- added copper zone on F.Cu, net GNDA
- added copper zone on In1.Cu, net GNDA
- added copper zone on In2.Cu, net GNDA
Other:
- board text added: "GND 24V0 GND ~{SYNC} SDO SDI SCLK 2B4 2B3 2B2 2B1 1B4 1B3 1B2 1B1 GND 3V3 GND GND -15V0 GND GND 5V0 GND SCL SDA GND GND DO_VDD GND GND 14V5 GND"

Commit message: backup
Parts:
- J1: renamed from J4; value CLP-133-02-G-D-BE -> FW-35-03-G-D-085-155; footprint connector_footprints:CLP-133-02-G-D-BE -> connector_footprints:FW-35-03-G-D-085-155
- J2, J3, J5: value CLP-133-02-G-D-BE -> CLP-135-02-G-D-BE; footprint connector_footprints:CLP-133-02-G-D-BE -> connector_footprints:CLP-135-02-G-D-BE
- J4: renamed from J1; value FW-33-03-G-D-085-155 -> CLP-135-02-G-D-BE; footprint connector_footprints:FW-33-03-G-D-085-155 -> connector_footprints:CLP-135-02-G-D-BE
- moved J1 31.3 mm to (139.7, 99.2)
- moved J4 31.3 mm to (139.7, 130.6)
Connections:
- J1 pad 53: GNDA -> unconnected-(J1-Pad53)
- J1 pad 54: GNDA -> unconnected-(J1-Pad54)
- J1 pad 55: GNDA -> unconnected-(J1-Pad55)
- J1 pad 56: GNDA -> unconnected-(J1-Pad56)
- J1 pad 57: /DO_VDD -> GNDA
- J1 pad 58: /DO_VDD -> GNDA
- J1 pad 61: GNDA -> /DO_VDD
- J1 pad 62: GNDA -> /DO_VDD
- J1 pad 63: /14V5 -> GNDA
- J1 pad 64: /14V5 -> GNDA
- J2 pad 57: /DO_VDD -> GNDA
- J2 pad 58: /DO_VDD -> GNDA
- J2 pad 61: GNDA -> /DO_VDD
- J2 pad 62: GNDA -> /DO_VDD
- J2 pad 63: /14V5 -> GNDA
- J2 pad 64: /14V5 -> GNDA
- J3 pad 55: GNDA -> unconnected-(J3-Pad55)
- J3 pad 56: GNDA -> unconnected-(J3-Pad56)
- J3 pad 57: /DO_VDD -> GNDA
- J3 pad 58: /DO_VDD -> GNDA
- J3 pad 61: GNDA -> /DO_VDD
- J3 pad 62: GNDA -> /DO_VDD
- J3 pad 63: /14V5 -> GNDA
- J3 pad 64: /14V5 -> GNDA
- J4 pad 53: GNDA -> unconnected-(J4-Pad53)
- J4 pad 54: GNDA -> unconnected-(J4-Pad54)
- J4 pad 57: /DO_VDD -> GNDA
- J4 pad 58: /DO_VDD -> GNDA
- J4 pad 61: GNDA -> /DO_VDD
- J4 pad 62: GNDA -> /DO_VDD
- J4 pad 63: /14V5 -> GNDA
- J4 pad 64: /14V5 -> GNDA
- J5 pad 53: GNDA -> unconnected-(J5-Pad53)
- J5 pad 54: GNDA -> unconnected-(J5-Pad54)
- J5 pad 55: GNDA -> unconnected-(J5-Pad55)
- J5 pad 56: GNDA -> unconnected-(J5-Pad56)
- J5 pad 57: /DO_VDD -> GNDA
- J5 pad 58: /DO_VDD -> GNDA
- J5 pad 61: GNDA -> /DO_VDD
- J5 pad 62: GNDA -> /DO_VDD
- J5 pad 63: /14V5 -> GNDA
- J5 pad 64: /14V5 -> GNDA
Routing:
- net GNDA: vias 104 -> 112
Other:
- board size 45.7 x 53.3 mm -> 48.3 x 53.3 mm
- board text added: "GND 24V0 GND ~{SYNC} SDO SDI SCLK 2B4 2B3 2B2 2B1 1B4 1B3 1B2 1B1 GND 3V3 GND GND -15V0 GND GND 5V0 GND SCL SDA AD0 AD1 GND GND DO_VDD GND GND 14V5 GND"
- board text removed: "GND 24V0 GND ~{SYNC} SDO SDI SCLK 2B4 2B3 2B2 2B1 1B4 1B3 1B2 1B1 GND 3V3 GND GND -15V0 GND GND 5V0 GND SCL SDA GND GND DO_VDD GND GND 14V5 GND"
