File: minimal_ad74416h_stack_adapter/minimal_ad74416h_stack_adapter.kicad_pcb (KiCad board)
At the start: 4 copper layers, 48.3 x 53.3 mm, 5 parts, among them J1 FW-35-03-G-D-085-155, J2 CLP-135-02-G-D-BE, J3 CLP-135-02-G-D-BE, J4 CLP-135-02-G-D-BE, J5 CLP-135-02-G-D-BE

Commit message: backup
Parts:
- moved J5 2.67 mm to (139.7, 140.1)
- moved J4 1.78 mm to (139.7, 128.8)
- moved J3 0.89 mm to (139.7, 117.5)
Routing:
- net /SDA: track 60.7 -> 58.0 mm
- net /~{SYNC}: track 60.7 -> 58.0 mm
- net /1B4: track 60.7 -> 58.0 mm
- net /SDO: track 60.7 -> 58.0 mm
- net /SDI: track 60.7 -> 58.0 mm
- net /SCLK: track 60.7 -> 58.0 mm
- net /2B4: track 60.7 -> 58.0 mm
- net /2B3: track 60.7 -> 58.0 mm
- net /2B1: track 60.7 -> 58.0 mm
- net /1B3: track 60.7 -> 58.0 mm
- net /1B2: track 60.7 -> 58.0 mm
- net /1B1: track 60.7 -> 58.0 mm
- net /SCL: track 60.7 -> 58.0 mm
- net /2B2: track 60.6 -> 58.0 mm
Other:
- board size 48.3 x 53.3 mm -> 48.3 x 50.7 mm

Commit message: backup
Parts:
- J1: value FW-35-03-G-D-085-155 -> FTSH-135-04-L-D; footprint connector_footprints:FW-35-03-G-D-085-155 -> connector_footprints:FTSH-135-04-L-D
- moved J1 2.00 mm to (139.7, 101.2)
Routing:
- net /SDI: track 58.0 -> 54.6 mm
- net /~{SYNC}: track 58.0 -> 54.6 mm
- net /SDO: track 58.0 -> 54.6 mm
- net /SDA: track 58.0 -> 54.6 mm
- net /SCLK: track 58.0 -> 54.6 mm
- net /SCL: track 58.0 -> 54.6 mm
- net /2B4: track 58.0 -> 54.6 mm
- net /2B3: track 58.0 -> 54.6 mm
- net /2B1: track 58.0 -> 54.6 mm
- net /1B4: track 58.0 -> 54.6 mm
- net /1B3: track 58.0 -> 54.6 mm
- net /1B2: track 58.0 -> 54.6 mm
- net /1B1: track 58.0 -> 54.6 mm
- net /2B2: track 58.0 -> 54.6 mm
Other:
- board size 48.3 x 50.7 mm -> 48.3 x 46.2 mm
